Commit message: feat: tacto enabled urdf

File: assets/leap_hand/digit_leap.urdf (robot description, URDF)
Before this commit: robot onshape, 17 links, 16 joints
Joints:
- joint 11: axis 0 0 -1 -> 0 1 0; origin xyz=9.7144514654701197287e-17 -0.036099999999999868305 0.00020000000000007511769 rpy=4.5935029425113685044e-17 -2.8730071914463799514e-16 1.5565411607615035382e-32 -> xyz=0.00628642410853349623 -0.041142383865420008027 0.014499999999999495931 rpy=1.57079632679 3.14159265359 1.4408183216511868558e-31
- joint 3: axis 0 0 -1 -> 0 1 0; origin xyz=-4.0880582495572692636e-09 -0.036100004210367367397 0.00020000000000007858714 rpy=4.5935029425113685044e-17 -2.8730071914463794583e-16 4.4395481053923607589e-32 -> xyz=0.00628642410853349623 -0.041142383865420008027 0.014499999999999495931 rpy=1.57079632679 3.14159265359 1.4408183216511868558e-31
- joint 7: axis 0 0 -1 -> 0 1 0; origin xyz=1.0061396160665481148e-16 -0.036099999999999854428 0.00020000000000007858714 rpy=4.5935029425113654229e-17 -2.8730071914463794583e-16 1.4408183216511868558e-31 -> xyz=0.00628642410853349623 -0.041142383865420008027 0.014499999999999495931 rpy=1.57079632679 3.14159265359 1.4408183216511868558e-31
