Commit message: feat: digit_leap

File: assets/leap_hand_thumb/digit_leap.urdf (robot description, URDF)
Before this commit: robot onshape, 17 links, 16 joints
Links:
- added link jig_finger, mass 0.016; collision mesh filename=JIG_finger.stl scale=0.001 0.001 0.001; visual mesh filename=JIG_finger.stl scale=0.001 0.001 0.001
- added link jig_finger_2, mass 0.016; collision mesh filename=JIG_finger.stl scale=0.001 0.001 0.001; visual mesh filename=JIG_finger.stl scale=0.001 0.001 0.001
- added link jig_finger_3, mass 0.016; collision mesh filename=JIG_finger.stl scale=0.001 0.001 0.001; visual mesh filename=JIG_finger.stl scale=0.001 0.001 0.001
Joints:
- added joint 16: type revolute, parent dip_3, child jig_finger_3, origin xyz=0 -0.036 0.015 rpy=0 0 -3.14159265359, axis 0 0 -1, limit lower=-0.506 upper=1.885 effort=0.95 velocity=8.48
- added joint 17: type revolute, parent dip_2, child jig_finger_2, origin xyz=0 -0.036 0.015 rpy=0 0 -3.14159265359, axis 0 0 1, limit lower=-0.506 upper=1.885 effort=0.95 velocity=8.48
- added joint 18: type revolute, parent dip, child jig_finger, origin xyz=0 -0.036 0.015 rpy=0 0 -3.14159265359, axis 0 0 1, limit lower=-0.506 upper=1.885 effort=0.95 velocity=8.48
- joint 11: axis 0 1 0 -> 0 0 0; origin xyz=0.00628642410853349623 -0.041142383865420008027 0.014499999999999495931 rpy=1.57079632679 3.14159265359 1.4408183216511868558e-31 -> xyz=-0.00028642410853349623 0.0161142383865420008027 -0.0010499999999999495931 rpy=1.57079632679 3.14159265359 3.14159265359; parent dip_3 -> jig_finger_3
- joint 3: axis 0 1 0 -> 0 0 0; origin xyz=0.00628642410853349623 -0.041142383865420008027 0.014499999999999495931 rpy=1.57079632679 3.14159265359 1.4408183216511868558e-31 -> xyz=-0.00028642410853349623 0.0161142383865420008027 -0.0010499999999999495931 rpy=1.57079632679 3.14159265359 3.1415926535; parent dip -> jig_finger
- joint 7: axis 0 1 0 -> 0 0 0; origin xyz=0.00628642410853349623 -0.041142383865420008027 0.014499999999999495931 rpy=1.57079632679 3.14159265359 1.4408183216511868558e-31 -> xyz=-0.00028642410853349623 0.0161142383865420008027 -0.0010499999999999495931 rpy=1.57079632679 3.14159265359 3.14159265359; parent dip_2 -> jig_finger_2
